Commit message: update 2021 06 21 .

File: humic_description/urdf/humic.urdf.xacro (robot description, xacro)
@@ -228,8 +228,8 @@
     <joint name="inner_column_joint" type="prismatic">
         <axis xyz="0 0 1" />
-        <limit velocity="0.01" effort="1000" lower="0" upper="0"/>
-        <origin xyz="0.135 0 0.25" rpy="0 0 0"/>
-        <!-- <limit velocity="0.01" effort="1000" lower="0" upper="0.50"/> -->
-        <!-- <origin xyz="0.135 0 0.05" rpy="0 0 0"/> -->
+	<!--<limit velocity="0.01" effort="1000" lower="0" upper="0"/>-->
+	<!--<origin xyz="0.135 0 0.25" rpy="0 0 0"/>-->
+        <limit velocity="0.01" effort="1000" lower="0" upper="0.50"/>
+        <origin xyz="0.135 0 0.05" rpy="0 0 0"/>
         <parent link="base_column_link"/>
         <child link="inner_column_link"/>
